Commit message: 优化urdf，优化坐标系

File: src/robot_urdf/urdf/robot.urdf (robot description, URDF)
Before this commit: robot robot_urdf, 12 links, 11 joints
Links:
- link base_link: mass 0.61343552337577 -> 2.0518821290605
- link link1: mass 1.76165867066071 -> None; geometry visual mesh filename=package://robot_urdf/meshes/L1.STL
- link link10: mass 0.397644492245874 -> None; geometry visual mesh filename=package://robot_urdf/meshes/L10.STL
- link link2: mass 2.02840748446522 -> None; geometry visual mesh filename=package://robot_urdf/meshes/L2.STL
- link link3: mass 1.3132850053279 -> None; geometry visual mesh filename=package://robot_urdf/meshes/L3.STL
- link link4: mass 1.71574111556864 -> None; geometry visual mesh filename=package://robot_urdf/meshes/L4.STL
- link link5: mass 1.33531734347054 -> None; geometry visual mesh filename=package://robot_urdf/meshes/L5.STL
- link link6: mass 1.71877897950771 -> None; geometry visual mesh filename=package://robot_urdf/meshes/L6.STL
- link link7: mass 1.394 -> None; geometry visual mesh filename=package://robot_urdf/meshes/L7.STL
- link link8: mass 0.10894 -> None; geometry visual mesh filename=package://robot_urdf/meshes/L8.STL
- link link9: mass 0.3401168202357 -> None; geometry visual mesh filename=package://robot_urdf/meshes/L9.STL
Joints:
- joint joint1: axis 0 1 0 -> 0 0 1; origin xyz=0.027469822907858 -0.289405264220156 0 rpy=1.5707963267949 0 1.5707963267949 -> xyz=0 0 0.0105 rpy=0 0 0
- joint joint10: axis 0 1 0 -> 0 0 -1; origin xyz=0.0405997949588489 0.0509999999999952 0.0192914268342251 rpy=-1.66340666484801 1.12517093240157 -0.102566626437443 -> xyz=0 -0.03895 -0.045 rpy=-1.5708 0 3.1416
- joint joint2: axis 0 1 0 -> 0 0 1; origin xyz=0 0.115812449934297 0 rpy=-1.57079632679443 1.52665095895204 -3.14159265358932 -> xyz=0 0.0715 0.0735 rpy=1.5707963267949 -1.5707963267949 0
- joint joint3: axis 0 -1 0 -> 0 0 -1; origin xyz=-0.18997 0 0.0035357 rpy=0 -1.3996 3.1416 -> xyz=0 -0.19 -0.01 rpy=0 0 1.5707963267949
- joint joint4: axis 0 1 0 -> 0 0 -1; origin xyz=0 0 0 rpy=2.56596813108925 1.25242393585874 1.0184622379495 -> xyz=0 0.0545 0.08 rpy=1.57079632679489 -1.5707963267949 0
- joint joint5: axis 0 -1 0 -> 0 0 -1; origin xyz=0.0946351936209319 0.210533090172604 -0.0762866795769143 rpy=2.28039917097598 -0.763007747213142 -1.53406250139247 -> xyz=0 0.127763139720814 -0.153153810567666 rpy=2.09439510239319 0 0
- joint joint6: axis 0 1 0 -> 0 0.5 0.8660254; origin xyz=0.0148674067720644 0.106324927585297 -0.059559132727178 rpy=1.76122232777038 0.543874247010192 2.3245839175662 -> xyz=0 -0.0926744834794736 0.0940194913397212 rpy=-0.523598775598299 0 0
- joint joint7: axis 0 1 0 -> 0 0 -1; origin xyz=0.0554883725781824 0 0.26321481817828 rpy=3.14159265358979 1.35917882149054 -3.14159265358979 -> xyz=0 -0.226210833618015 0.146191342951089 rpy=2.6179938779915 0 0
- joint joint8: axis 0 1 0 -> 0 0 -1; origin xyz=-0.167648757864712 0.046872009089088 -0.000645357590316559 rpy=1.57079632679201 -1.56694688340607 -3.14159265358691 -> xyz=0 0.1684 -0.070356758575594 rpy=1.5707963267949 0 0
- joint joint9: axis 0 1 0 -> 0 0 -1; origin xyz=0 -0.0760000000000005 -0.0507999999999832 rpy=1.5707963267949 0 -2.69801321173957 -> xyz=0 0.045657 -0.07525 rpy=1.5708 -1.5708 0
- joint world_to_base: origin xyz=0 0 0 rpy=-1.57079632679 0 0 -> xyz=0 0 0 rpy=0 0 0

Commit message: 修改5、6轴方向

File: src/robot_urdf/urdf/robot.urdf (robot description, URDF)
Before this commit: robot robot_urdf, 14 links, 13 joints
Joints:
- joint joint6: axis 0 0 1 -> 0 0 -1

File: src/upperlimb_robot/urdf/left_arm_experiment.urdf (robot description, URDF)
Before this commit: robot robot_urdf, 14 links, 13 joints
Joints:
- joint joint6: axis 0 0 1 -> 0 0 -1
