Commit message: 修改urdf模型，修改正逆运动学计算，修改rviz显示

File: src/pinocchio_kin_demo/urdf/my_robot.urdf (robot description, URDF)
Before this commit: robot robot_urdf, 12 links, 11 joints
Links:
- link link1: mass None -> 1.76165866952677; geometry collision mesh filename=package://robot_urdf/meshes/link1.STL; visual mesh filename=package://robot_urdf/meshes/link1.STL
- link link10: mass None -> 0.117868082328721; geometry collision mesh filename=package://robot_urdf/meshes/link10.STL; visual mesh filename=package://robot_urdf/meshes/link10.STL
- link link2: mass None -> 1.59468357316661; geometry collision mesh filename=package://robot_urdf/meshes/link2.STL; visual mesh filename=package://robot_urdf/meshes/link2.STL
- link link3: mass None -> 1.50899705647033; geometry collision mesh filename=package://robot_urdf/meshes/link3.STL; visual mesh filename=package://robot_urdf/meshes/link3.STL
- link link4: mass None -> 1.52002906360623; geometry collision mesh filename=package://robot_urdf/meshes/link4.STL; visual mesh filename=package://robot_urdf/meshes/link4.STL
- link link5: mass None -> 1.33531731957906; geometry collision mesh filename=package://robot_urdf/meshes/link5.STL; visual mesh filename=package://robot_urdf/meshes/link5.STL
- link link6: mass None -> 1.59319846120862; geometry collision mesh filename=package://robot_urdf/meshes/link6.STL; visual mesh filename=package://robot_urdf/meshes/link6.STL
- link link7: mass None -> 0.53340488284912; geometry collision mesh filename=package://robot_urdf/meshes/link7.STL; visual mesh filename=package://robot_urdf/meshes/link7.STL
- link link8: mass None -> 0.388714289768506; geometry collision mesh filename=package://robot_urdf/meshes/link8.STL; visual mesh filename=package://robot_urdf/meshes/link8.STL
- link link9: mass None -> 0.340116810823749; geometry collision mesh filename=package://robot_urdf/meshes/link9.STL; visual mesh filename=package://robot_urdf/meshes/link9.STL
Joints:
- removed joint world_to_base
- added joint world_to_base_link: type fixed, parent world, child base_link, origin xyz=0 0 0 rpy=1.5708 0 0
- joint joint1: axis 0 0 1 -> 0 0 -1; limit lower=-1.57079632679 upper=1.57079632679 effort=100.0 velocity=2.0 -> lower=-3.1416 upper=3.1416 effort=50 velocity=2.0; origin xyz=0 0 0.0105 rpy=0 0 0 -> xyz=0 0 0 rpy=0 0 -1.5707963267949
- joint joint10: axis 0 0 -1 -> (none); limit lower=-1.57079632679 upper=1.57079632679 effort=100.0 velocity=2.0 -> (none); origin xyz=0 -0.03895 -0.045 rpy=-1.5708 0 3.1416 -> xyz=0.0449499999999999 0 -0.0509999999999973 rpy=-1.5707963267949 0 -1.57079632679491; type revolute -> fixed
- joint joint2: axis 0 0 1 -> 0 0 -1; limit lower=-1.57079632679 upper=1.57079632679 effort=100.0 velocity=2.0 -> lower=-3.1416 upper=3.1416 effort=50 velocity=2.0; origin xyz=0 0.0715 0.0735 rpy=1.5707963267949 -1.5707963267949 0 -> xyz=0.0715 0 -0.0735000000000018 rpy=-1.5707963267949 0 1.5707963267949
- joint joint3: axis 0 0 -1 -> 0 0 1; limit lower=-1.57079632679 upper=1.57079632679 effort=100.0 velocity=2.0 -> lower=-3.1416 upper=3.1416 effort=50 velocity=2.0; origin xyz=0 -0.19 -0.01 rpy=0 0 1.5707963267949 -> xyz=0.19 0 -0.01 rpy=-3.14159265358979 0 -1.57079632679489
- joint joint4: axis 0 0 -1 -> 0 0 1; limit lower=-1.57079632679 upper=1.57079632679 effort=100.0 velocity=2.0 -> lower=-3.1416 upper=3.1416 effort=50 velocity=2.0; origin xyz=0 0.0545 0.08 rpy=1.57079632679489 -1.5707963267949 0 -> xyz=0.0545000000000001 0 -0.08 rpy=3.14159265358979 1.5707963267949 0
- joint joint5: limit lower=-1.57079632679 upper=1.57079632679 effort=100.0 velocity=2.0 -> lower=-3.1416 upper=3.1416 effort=50 velocity=2.0; origin xyz=0 0.127763139720814 -0.153153810567666 rpy=2.09439510239319 0 0 -> xyz=0.127763139720814 0 -0.153153810567666 rpy=-2.09439510239319 0 1.5707963267949
- joint joint6: axis 0 0.5 0.8660254 -> 0 0 1; limit lower=-1.57079632679 upper=1.57079632679 effort=100.0 velocity=2.0 -> lower=-3.1416 upper=3.1416 effort=50 velocity=2.0; origin xyz=0 -0.0926744834794736 0.0940194913397212 rpy=-0.523598775598299 0 0 -> xyz=0.0926744834794751 0 0.0940194913397204 rpy=-2.25551552979719 -0.65905803582641 -1.10714871779409
- joint joint7: axis 0 0 -1 -> 0 0 1; limit lower=-1.57079632679 upper=1.57079632679 effort=100.0 velocity=2.0 -> lower=-3.1416 upper=3.1416 effort=50 velocity=2.0; origin xyz=0 -0.226210833618015 0.146191342951089 rpy=2.6179938779915 0 0 -> xyz=0.269 0 -0.008 rpy=0 0 0
- joint joint8: axis 0 0 -1 -> (none); limit lower=-1.57079632679 upper=1.57079632679 effort=100.0 velocity=2.0 -> (none); origin xyz=0 0.1684 -0.070356758575594 rpy=1.5707963267949 0 0 -> xyz=0.18565 0 -0.075 rpy=-1.5708 0 1.5708; type revolute -> fixed
- joint joint9: axis 0 0 -1 -> (none); limit lower=-1.57079632679 upper=1.57079632679 effort=100.0 velocity=2.0 -> (none); origin xyz=0 0.045657 -0.07525 rpy=1.5708 -1.5708 0 -> xyz=0 -0.0508 -0.058 rpy=1.5708 0 0; type revolute -> fixed

File: src/robot_urdf/urdf/fixrobot.urdf (robot description, URDF)
Before this commit: robot robot_urdf, 12 links, 11 joints
Links:
- link link1: geometry collision mesh filename=package://robot_urdf/meshes/link1.STL; visual mesh filename=package://robot_urdf/meshes/link1.STL
- link link10: mass 0.118059085282791 -> 0.117868082328721; geometry collision mesh filename=package://robot_urdf/meshes/link10.STL; visual mesh filename=package://robot_urdf/meshes/link10.STL
- link link2: geometry collision mesh filename=package://robot_urdf/meshes/link2.STL; visual mesh filename=package://robot_urdf/meshes/link2.STL
- link link3: geometry collision mesh filename=package://robot_urdf/meshes/link3.STL; visual mesh filename=package://robot_urdf/meshes/link3.STL
- link link4: mass 1.52002907368431 -> 1.52002906360623; geometry collision mesh filename=package://robot_urdf/meshes/link4.STL; visual mesh filename=package://robot_urdf/meshes/link4.STL
- link link5: mass 1.33531721897832 -> 1.33531731957906; geometry collision mesh filename=package://robot_urdf/meshes/link5.STL; visual mesh filename=package://robot_urdf/meshes/link5.STL
- link link6: mass 1.57384762218888 -> 1.59319846120862; geometry collision mesh filename=package://robot_urdf/meshes/link6.STL; visual mesh filename=package://robot_urdf/meshes/link6.STL
- link link7: mass 0.533993935665024 -> 0.53340488284912; geometry collision mesh filename=package://robot_urdf/meshes/link7.STL; visual mesh filename=package://robot_urdf/meshes/link7.STL
- link link8: mass 0.388251678654185 -> 0.388714289768506; geometry collision mesh filename=package://robot_urdf/meshes/link8.STL; visual mesh filename=package://robot_urdf/meshes/link8.STL
- link link9: mass 0.340116805099853 -> 0.340116810823749; geometry collision mesh filename=package://robot_urdf/meshes/link9.STL; visual mesh filename=package://robot_urdf/meshes/link9.STL
Joints:
- removed joint world_to_base
- added joint world_to_base_link: type fixed, parent world, child base_link, origin xyz=0 0 0 rpy=1.5708 0 0
- joint joint1: axis 0 0 1 -> 0 0 -1; limit (none) -> lower=-3.1416 upper=3.1416 effort=50 velocity=2.0; origin xyz=0 0 0.0105 rpy=0 0 0 -> xyz=0 0 0 rpy=0 0 -1.5707963267949; type continuous -> revolute
- joint joint10: origin xyz=0 -0.03895 -0.045 rpy=-1.5708 0 3.1416 -> xyz=0.0449499999999999 0 -0.0509999999999973 rpy=-1.5707963267949 0 -1.57079632679491
- joint joint2: axis 0 0 1 -> 0 0 -1; limit (none) -> lower=-3.1416 upper=3.1416 effort=50 velocity=2.0; origin xyz=0 0.0715 0.0735 rpy=1.5707963267949 -1.5707963267949 0 -> xyz=0.0715 0 -0.0735000000000018 rpy=-1.5707963267949 0 1.5707963267949; type continuous -> revolute
- joint joint3: axis 0 0 -1 -> 0 0 1; limit (none) -> lower=-3.1416 upper=3.1416 effort=50 velocity=2.0; origin xyz=0 -0.19 -0.01 rpy=0 0 1.5707963267949 -> xyz=0.19 0 -0.01 rpy=-3.14159265358979 0 -1.57079632679489; type continuous -> revolute
- joint joint4: axis 0 0 -1 -> 0 0 1; limit (none) -> lower=-3.1416 upper=3.1416 effort=50 velocity=2.0; origin xyz=0 0.0545 0.08 rpy=1.57079632679489 -1.5707963267949 0 -> xyz=0.0545000000000001 0 -0.08 rpy=3.14159265358979 1.5707963267949 0; type continuous -> revolute
- joint joint5: limit (none) -> lower=-3.1416 upper=3.1416 effort=50 velocity=2.0; origin xyz=0 0.127763139720814 -0.153153810567666 rpy=2.09439510239319 0 0 -> xyz=0.127763139720814 0 -0.153153810567666 rpy=-2.09439510239319 0 1.5707963267949; type continuous -> revolute
- joint joint6: axis 0 0.5 0.8660254 -> 0 0 1; limit (none) -> lower=-3.1416 upper=3.1416 effort=50 velocity=2.0; origin xyz=0 -0.0926744834794736 0.0940194913397212 rpy=-0.523598775598299 0 0 -> xyz=0.0926744834794751 0 0.0940194913397204 rpy=-2.25551552979719 -0.65905803582641 -1.10714871779409; type continuous -> revolute
- joint joint7: axis (none) -> 0 0 1; limit (none) -> lower=-3.1416 upper=3.1416 effort=50 velocity=2.0; origin xyz=0 -0.226210833618015 0.146191342951089 rpy=2.6179938779915 0 0 -> xyz=0.269 0 -0.008 rpy=0 0 0; type fixed -> revolute
- joint joint8: origin xyz=0 0.1684 -0.070356758575594 rpy=1.5707963267949 0 0 -> xyz=0.18565 0 -0.075 rpy=-1.5708 0 1.5708
- joint joint9: origin xyz=0 0.045657 -0.07525 rpy=1.5708 -1.5708 0 -> xyz=0 -0.0508 -0.058 rpy=1.5708 0 0

File: src/robot_urdf/urdf/robot.urdf (robot description, URDF)
Before this commit: robot robot_urdf, 12 links, 11 joints
Links:
- link link1: mass None -> 1.76165866952677; geometry collision mesh filename=package://robot_urdf/meshes/link1.STL; visual mesh filename=package://robot_urdf/meshes/link1.STL
- link link10: mass None -> 0.117868082328721; geometry collision mesh filename=package://robot_urdf/meshes/link10.STL; visual mesh filename=package://robot_urdf/meshes/link10.STL
- link link2: mass None -> 1.59468357316661; geometry collision mesh filename=package://robot_urdf/meshes/link2.STL; visual mesh filename=package://robot_urdf/meshes/link2.STL
- link link3: mass None -> 1.50899705647033; geometry collision mesh filename=package://robot_urdf/meshes/link3.STL; visual mesh filename=package://robot_urdf/meshes/link3.STL
- link link4: mass None -> 1.52002906360623; geometry collision mesh filename=package://robot_urdf/meshes/link4.STL; visual mesh filename=package://robot_urdf/meshes/link4.STL
- link link5: mass None -> 1.33531731957906; geometry collision mesh filename=package://robot_urdf/meshes/link5.STL; visual mesh filename=package://robot_urdf/meshes/link5.STL
- link link6: mass None -> 1.59319846120862; geometry collision mesh filename=package://robot_urdf/meshes/link6.STL; visual mesh filename=package://robot_urdf/meshes/link6.STL
- link link7: mass None -> 0.53340488284912; geometry collision mesh filename=package://robot_urdf/meshes/link7.STL; visual mesh filename=package://robot_urdf/meshes/link7.STL
- link link8: mass None -> 0.388714289768506; geometry collision mesh filename=package://robot_urdf/meshes/link8.STL; visual mesh filename=package://robot_urdf/meshes/link8.STL
- link link9: mass None -> 0.340116810823749; geometry collision mesh filename=package://robot_urdf/meshes/link9.STL; visual mesh filename=package://robot_urdf/meshes/link9.STL
Joints:
- removed joint world_to_base
- added joint world_to_base_link: type fixed, parent world, child base_link, origin xyz=0 0 0 rpy=1.5708 0 0
- joint joint1: axis 0 0 1 -> 0 0 -1; limit (none) -> lower=-3.1416 upper=3.1416 effort=50 velocity=2.0; origin xyz=0 0 0.0105 rpy=0 0 0 -> xyz=0 0 0 rpy=0 0 -1.5707963267949; type continuous -> revolute
- joint joint10: limit (none) -> lower=-3.1416 upper=3.1416 effort=50 velocity=2.0; origin xyz=0 -0.03895 -0.045 rpy=-1.5708 0 3.1416 -> xyz=0.0449499999999999 0 -0.0509999999999973 rpy=-1.5707963267949 0 -1.57079632679491; type continuous -> revolute
- joint joint2: axis 0 0 1 -> 0 0 -1; limit (none) -> lower=-3.1416 upper=3.1416 effort=50 velocity=2.0; origin xyz=0 0.0715 0.0735 rpy=1.5707963267949 -1.5707963267949 0 -> xyz=0.0715 0 -0.0735000000000018 rpy=-1.5707963267949 0 1.5707963267949; type continuous -> revolute
- joint joint3: axis 0 0 -1 -> 0 0 1; limit (none) -> lower=-3.1416 upper=3.1416 effort=50 velocity=2.0; origin xyz=0 -0.19 -0.01 rpy=0 0 1.5707963267949 -> xyz=0.19 0 -0.01 rpy=-3.14159265358979 0 -1.57079632679489; type continuous -> revolute
- joint joint4: axis 0 0 -1 -> 0 0 1; limit (none) -> lower=-3.1416 upper=3.1416 effort=50 velocity=2.0; origin xyz=0 0.0545 0.08 rpy=1.57079632679489 -1.5707963267949 0 -> xyz=0.0545000000000001 0 -0.08 rpy=3.14159265358979 1.5707963267949 0; type continuous -> revolute
- joint joint5: limit (none) -> lower=-3.1416 upper=3.1416 effort=50 velocity=2.0; origin xyz=0 0.127763139720814 -0.153153810567666 rpy=2.09439510239319 0 0 -> xyz=0.127763139720814 0 -0.153153810567666 rpy=-2.09439510239319 0 1.5707963267949; type continuous -> revolute
- joint joint6: axis 0 0.5 0.8660254 -> 0 0 1; limit (none) -> lower=-3.1416 upper=3.1416 effort=50 velocity=2.0; origin xyz=0 -0.0926744834794736 0.0940194913397212 rpy=-0.523598775598299 0 0 -> xyz=0.0926744834794751 0 0.0940194913397204 rpy=-2.25551552979719 -0.65905803582641 -1.10714871779409; type continuous -> revolute
- joint joint7: axis 0 0 -1 -> 0 0 1; limit (none) -> lower=-3.1416 upper=3.1416 effort=50 velocity=2.0; origin xyz=0 -0.226210833618015 0.146191342951089 rpy=2.6179938779915 0 0 -> xyz=0.269 0 -0.008 rpy=0 0 0; type continuous -> revolute
- joint joint8: limit (none) -> lower=-3.1416 upper=3.1416 effort=50 velocity=2.0; origin xyz=0 0.1684 -0.070356758575594 rpy=1.5707963267949 0 0 -> xyz=0.18565 0 -0.075 rpy=-1.5708 0 1.5708; type continuous -> revolute
- joint joint9: limit (none) -> lower=-3.1416 upper=3.1416 effort=50 velocity=2.0; origin xyz=0 0.045657 -0.07525 rpy=1.5708 -1.5708 0 -> xyz=0 -0.0508 -0.058 rpy=1.5708 0 0; type continuous -> revolute

Commit message: 修改urdf模型，与代码中起始位置对应；增加力传感器坐标及标记点

File: src/pinocchio_kin_demo/urdf/my_robot.urdf (robot description, URDF)
Before this commit: robot urdfv4, 12 links, 11 joints
Links:
- added link ft_sensor_frame; visual sphere radius=0.01
- link base_link: mass 2.0518821290605 -> None; geometry visual mesh filename=package://robot_urdf/meshes/base_link.STL
- link link1: mass 1.76165866952677 -> None; geometry visual mesh filename=package://robot_urdf/meshes/link1.STL
- link link10: mass 0.117868082328721 -> None; geometry visual mesh filename=package://robot_urdf/meshes/link10.STL
- link link2: mass 1.59468357316661 -> None; geometry visual mesh filename=package://robot_urdf/meshes/link2.STL
- link link3: mass 1.50899705647033 -> None; geometry visual mesh filename=package://robot_urdf/meshes/link3.STL
- link link4: mass 1.52002906360623 -> None; geometry visual mesh filename=package://robot_urdf/meshes/link4.STL
- link link5: mass 1.33531731957906 -> None; geometry visual mesh filename=package://robot_urdf/meshes/link5.STL
- link link6: mass 1.59319846120862 -> None; geometry visual mesh filename=package://robot_urdf/meshes/link6.STL
- link link7: mass 0.53340488284912 -> None; geometry visual mesh filename=package://robot_urdf/meshes/link7.STL
- link link8: mass 0.388714289768506 -> None; geometry visual mesh filename=package://robot_urdf/meshes/link8.STL
- link link9: mass 0.340116810823749 -> None; geometry visual mesh filename=package://robot_urdf/meshes/link9.STL
Joints:
- added joint ft_sensor_joint: type fixed, parent link6, child ft_sensor_frame, origin xyz=0.18416 0 -0.01731 rpy=3.1351 0 -1.5708
- joint joint1: limit lower=-3.1416 upper=3.1416 effort=50 velocity=2.0 -> lower=-3.1416 upper=3.1416 effort=50 velocity=2; origin xyz=0 0 0 rpy=0 0 -1.5707963267949 -> xyz=0 0 0 rpy=0 0 -1.5708
- joint joint10: origin xyz=0.0449499999999999 0 -0.0509999999999973 rpy=-1.5707963267949 0 -1.57079632679491 -> xyz=-0.04495 0 -0.051 rpy=-1.5708 -0.01414 1.5708
- joint joint2: limit lower=-3.1416 upper=3.1416 effort=50 velocity=2.0 -> lower=-3.1416 upper=3.1416 effort=50 velocity=2; origin xyz=0.0715 0 -0.0735000000000018 rpy=-1.5707963267949 0 1.5707963267949 -> xyz=0.0715 0 -0.0735 rpy=-1.5708 0 1.5708
- joint joint3: limit lower=-3.1416 upper=3.1416 effort=50 velocity=2.0 -> lower=-3.1416 upper=3.1416 effort=50 velocity=2; origin xyz=0.19 0 -0.01 rpy=-3.14159265358979 0 -1.57079632679489 -> xyz=0.19 0 -0.01 rpy=-3.1416 0 -1.5708
- joint joint4: limit lower=-3.1416 upper=3.1416 effort=50 velocity=2.0 -> lower=-3.1416 upper=3.1416 effort=50 velocity=2; origin xyz=0.0545000000000001 0 -0.08 rpy=3.14159265358979 1.5707963267949 0 -> xyz=0.0545 0 -0.08 rpy=1.5708 0.95993 -1.5708
- joint joint5: limit lower=-3.1416 upper=3.1416 effort=50 velocity=2.0 -> lower=-3.1416 upper=3.1416 effort=50 velocity=2; origin xyz=0.127763139720814 0 -0.153153810567666 rpy=-2.09439510239319 0 1.5707963267949 -> xyz=0.12776 0 -0.15315 rpy=-2.1198 0.29022 1.3975
- joint joint6: limit lower=-3.1416 upper=3.1416 effort=50 velocity=2.0 -> lower=-3.1416 upper=3.1416 effort=50 velocity=2; origin xyz=0.0926744834794751 0 0.0940194913397204 rpy=-2.25551552979719 -0.65905803582641 -1.10714871779409 -> xyz=0.092667 0.0011397 0.094019 rpy=-2.3595 -0.78866 -0.93839
- joint joint7: limit lower=-3.1416 upper=3.1416 effort=50 velocity=2.0 -> lower=-3.1416 upper=3.1416 effort=50 velocity=2; origin xyz=0.269 0 -0.008 rpy=0 0 0 -> xyz=0.269 0 -0.008
- joint joint9: origin xyz=0 -0.0508 -0.058 rpy=1.5708 0 0 -> xyz=0 -0.0508 -0.058 rpy=-1.5708 0 -3.1416

File: src/robot_urdf/urdf/robot.urdf (robot description, URDF)
Before this commit: robot urdfv4, 12 links, 11 joints
Links:
- added link ft_sensor_frame; visual sphere radius=0.01
- link base_link: mass 2.0518821290605 -> None; geometry visual mesh filename=package://robot_urdf/meshes/base_link.STL
- link link1: mass 1.76165866952677 -> None; geometry visual mesh filename=package://robot_urdf/meshes/link1.STL
- link link10: mass 0.117868082328721 -> None; geometry visual mesh filename=package://robot_urdf/meshes/link10.STL
- link link2: mass 1.59468357316661 -> None; geometry visual mesh filename=package://robot_urdf/meshes/link2.STL
- link link3: mass 1.50899705647033 -> None; geometry visual mesh filename=package://robot_urdf/meshes/link3.STL
- link link4: mass 1.52002906360623 -> None; geometry visual mesh filename=package://robot_urdf/meshes/link4.STL
- link link5: mass 1.33531731957906 -> None; geometry visual mesh filename=package://robot_urdf/meshes/link5.STL
- link link6: mass 1.59319846120862 -> None; geometry visual mesh filename=package://robot_urdf/meshes/link6.STL
- link link7: mass 0.53340488284912 -> None; geometry visual mesh filename=package://robot_urdf/meshes/link7.STL
- link link8: mass 0.388714289768506 -> None; geometry visual mesh filename=package://robot_urdf/meshes/link8.STL
- link link9: mass 0.340116810823749 -> None; geometry visual mesh filename=package://robot_urdf/meshes/link9.STL
Joints:
- added joint ft_sensor_joint: type fixed, parent link6, child ft_sensor_frame, origin xyz=0.18416 0 -0.01731 rpy=3.1351 0 -1.5708
- joint joint1: limit lower=-3.1416 upper=3.1416 effort=50 velocity=2.0 -> lower=-3.1416 upper=3.1416 effort=50 velocity=2; origin xyz=0 0 0 rpy=0 0 -1.5707963267949 -> xyz=0 0 0 rpy=0 0 -1.5708
- joint joint10: limit lower=-3.1416 upper=3.1416 effort=50 velocity=2.0 -> lower=-3.1416 upper=3.1416 effort=50 velocity=2; origin xyz=0.0449499999999999 0 -0.0509999999999973 rpy=-1.5707963267949 0 -1.57079632679491 -> xyz=-0.04495 0 -0.051 rpy=-1.5708 -0.01414 1.5708
- joint joint2: limit lower=-3.1416 upper=3.1416 effort=50 velocity=2.0 -> lower=-3.1416 upper=3.1416 effort=50 velocity=2; origin xyz=0.0715 0 -0.0735000000000018 rpy=-1.5707963267949 0 1.5707963267949 -> xyz=0.0715 0 -0.0735 rpy=-1.5708 0 1.5708
- joint joint3: limit lower=-3.1416 upper=3.1416 effort=50 velocity=2.0 -> lower=-3.1416 upper=3.1416 effort=50 velocity=2; origin xyz=0.19 0 -0.01 rpy=-3.14159265358979 0 -1.57079632679489 -> xyz=0.19 0 -0.01 rpy=-3.1416 0 -1.5708
- joint joint4: limit lower=-3.1416 upper=3.1416 effort=50 velocity=2.0 -> lower=-3.1416 upper=3.1416 effort=50 velocity=2; origin xyz=0.0545000000000001 0 -0.08 rpy=3.14159265358979 1.5707963267949 0 -> xyz=0.0545 0 -0.08 rpy=1.5708 0.95993 -1.5708
- joint joint5: limit lower=-3.1416 upper=3.1416 effort=50 velocity=2.0 -> lower=-3.1416 upper=3.1416 effort=50 velocity=2; origin xyz=0.127763139720814 0 -0.153153810567666 rpy=-2.09439510239319 0 1.5707963267949 -> xyz=0.12776 0 -0.15315 rpy=-2.1198 0.29022 1.3975
- joint joint6: limit lower=-3.1416 upper=3.1416 effort=50 velocity=2.0 -> lower=-3.1416 upper=3.1416 effort=50 velocity=2; origin xyz=0.0926744834794751 0 0.0940194913397204 rpy=-2.25551552979719 -0.65905803582641 -1.10714871779409 -> xyz=0.092667 0.0011397 0.094019 rpy=-2.3595 -0.78866 -0.93839
- joint joint7: limit lower=-3.1416 upper=3.1416 effort=50 velocity=2.0 -> lower=-3.1416 upper=3.1416 effort=50 velocity=2; origin xyz=0.269 0 -0.008 rpy=0 0 0 -> xyz=0.269 0 -0.008
- joint joint8: limit lower=-3.1416 upper=3.1416 effort=50 velocity=2.0 -> lower=-3.1416 upper=3.1416 effort=50 velocity=2
- joint joint9: limit lower=-3.1416 upper=3.1416 effort=50 velocity=2.0 -> lower=-3.1416 upper=3.1416 effort=50 velocity=2; origin xyz=0 -0.0508 -0.058 rpy=1.5708 0 0 -> xyz=0 -0.0508 -0.058 rpy=-1.5708 0 -3.1416

Commit message: 修改偏置零位

File: src/pinocchio_kin_demo/urdf/my_robot.urdf (robot description, URDF)
Before this commit: robot robot_urdf, 13 links, 12 joints
Links:
- added link ft_sensor_frame_2; visual sphere radius=0.01
Joints:
- added joint ft_sensor_joint_2: type fixed, parent link10, child ft_sensor_frame_2, origin xyz=0.082 -0.0287 -0.06447  rpy=1.5643 -1.5225 1.5708

File: src/robot_urdf/urdf/robot.urdf (robot description, URDF)
Before this commit: robot robot_urdf, 13 links, 12 joints
Links:
- added link ft_sensor_frame_2; visual sphere radius=0.01
Joints:
- added joint ft_sensor_joint_2: type fixed, parent link10, child ft_sensor_frame_2, origin xyz=0.082 -0.0287 -0.06447  rpy=1.5643 -1.5225 1.5708
