Commit message: feat(urdf): 为机器人模型补充惯性参数（含 world 坐标系版本）
- 为所有连杆（base_link ~ link10）添加 inertial（质量、质心、惯量矩阵）
- 保持 SolidWorks 导出的惯性数据不变
- 将惯性信息集成到包含 world 坐标系的新 URDF 中
- 不修改原有运动学结构（包括 link8~10 的 fixed 关节）
- 确保惯性仍定义在各 link 局部坐标系下

说明：
- 引入 world 坐标系不会影响惯性参数的正确性
- 未改动 visual、joint 及 mesh 定义

---

feat(urdf): add inertial parameters to robot model with world frame

- Added inertial (mass, COM, inertia tensor) for all links (base_link ~ link10)
- Preserved original SolidWorks-exported inertial data
- Integrated inertial into updated URDF with world frame
- Kept kinematic structure unchanged (including fixed joints for link8~10)
- Ensured inertial definitions remain in link-local frames

Notes:
- Inertial frames are unaffected by world frame addition
- No modifications to visual, joint, or mesh definitions

File: src/pinocchio_kin_demo/urdf/my_robot.urdf (robot description, URDF)
Before this commit: robot robot_urdf, 14 links, 13 joints
Links:
- link base_link: mass None -> 2.0518821290605
- link link1: mass None -> 1.76165866952677
- link link10: mass None -> 0.118059114867053
- link link2: mass None -> 1.59468357316661
- link link3: mass None -> 1.50899705647033
- link link4: mass None -> 1.52002907684628
- link link5: mass None -> 1.33531733905559
- link link6: mass None -> 1.57403690632572
- link link7: mass None -> 0.53341444148306
- link link8: mass None -> 0.388714250535921
- link link9: mass None -> 0.340116837655435

File: src/robot_urdf/urdf/robot.urdf (robot description, URDF)
Before this commit: robot robot_urdf, 14 links, 13 joints
Links:
- link base_link: mass None -> 2.0518821290605
- link link1: mass None -> 1.76165866952677
- link link10: mass None -> 0.118059114867053
- link link2: mass None -> 1.59468357316661
- link link3: mass None -> 1.50899705647033
- link link4: mass None -> 1.52002907684628
- link link5: mass None -> 1.33531733905559
- link link6: mass None -> 1.57403690632572
- link link7: mass None -> 0.53341444148306
- link link8: mass None -> 0.388714250535921
- link link9: mass None -> 0.340116837655435

Commit message: refactor(control): 完善模式切换状态机与零偏校验，规范控制层注释；修正URDF中joint7的Z轴方向 / refactor(control): improve mode state machine and bias validation, standardize control layer comments; fix Z-axis direction of joint7 in URDF

File: src/pinocchio_kin_demo/urdf/my_robot.urdf (robot description, URDF)
Before this commit: robot robot_urdf, 14 links, 13 joints
Joints:
- joint joint7: axis 0 0 1 -> 0 0 -1

File: src/robot_urdf/urdf/robot.urdf (robot description, URDF)
Before this commit: robot robot_urdf, 14 links, 13 joints
Joints:
- joint joint7: axis 0 0 1 -> 0 0 -1

Commit message: 更新模型显示

File: src/pinocchio_kin_demo/urdf/my_robot.urdf (robot description, URDF)
Before this commit: robot robot_urdf, 14 links, 13 joints
Joints:
- joint ft_sensor_joint: origin xyz=0.18416 0 -0.01731 rpy=3.1351 0 -1.5708 -> xyz=0.18416 0 -0.01731 rpy=-3.1351 0 3.14159
- joint ft_sensor_joint_2: origin xyz=0.082 -0.0287 -0.06447  rpy=1.5643 -1.5225 1.5708 -> xyz=0.082 -0.0287 -0.06447  rpy=1.5708 0 3.14159

File: src/robot_urdf/urdf/fixrobot.urdf (robot description, URDF)
Before this commit: robot robot_urdf, 14 links, 13 joints
Joints:
- joint ft_sensor_joint: origin xyz=0.18416 0 -0.01731 rpy=3.1351 0 -1.5708 -> xyz=0.18416 0 -0.01731 rpy=-3.1351 0 3.14159
- joint ft_sensor_joint_2: origin xyz=0.082 -0.0287 -0.06447  rpy=1.5643 -1.5225 1.5708 -> xyz=0.082 -0.0287 -0.06447  rpy=1.5708 0 3.14159
- joint joint6: axis 0 0 1 -> 0 0 -1

File: src/robot_urdf/urdf/robot.urdf (robot description, URDF)
Before this commit: robot robot_urdf, 14 links, 13 joints
Joints:
- joint ft_sensor_joint: origin xyz=0.18416 0 -0.01731 rpy=3.1351 0 -1.5708 -> xyz=0.18416 0 -0.01731 rpy=-3.1351 0 3.14159
- joint ft_sensor_joint_2: origin xyz=0.082 -0.0287 -0.06447  rpy=1.5643 -1.5225 1.5708 -> xyz=0.082 -0.0287 -0.06447  rpy=1.5708 0 3.14159

File: src/upperlimb_robot/urdf/left_arm_experiment.urdf (robot description, URDF)
Before this commit: robot robot_urdf, 14 links, 13 joints
Joints:
- joint ft_sensor_joint: origin xyz=0.18416 0 -0.01731 rpy=3.1351 0 -1.5708 -> xyz=0.18416 0 -0.01731 rpy=-3.1351 0 3.14159
- joint ft_sensor_joint_2: origin xyz=0.082 -0.0287 -0.06447 rpy=1.5643 -1.5225 1.5708 -> xyz=0.082 -0.0287 -0.06447  rpy=1.5708 0 3.14159
