Commit message: feat:增加joint1/2/3为活动关节

File: src/upperlimb_robot/urdf/left_arm_experiment.urdf (robot description, URDF)
Before this commit: robot robot_urdf, 14 links, 13 joints
Joints:
- joint joint1: type fixed -> revolute
- joint joint2: type fixed -> revolute
- joint joint3: type fixed -> revolute

Commit message: feat:左臂2号关节方向修正

File: src/upperlimb_robot/urdf/left_arm_experiment.urdf (robot description, URDF)
Before this commit: robot robot_urdf, 14 links, 13 joints
Joints:
- joint joint2: axis 0 0 -1 -> 0 0 1
