Commit message: feat:模型修改与调整

File: src/upperlimb_robot/urdf/robot_arms.urdf (robot description, URDF)
Before this commit: robot robot_arms, 26 links, 25 joints
Joints:
- joint joint1: limit (none) -> lower=-3.1416 upper=3.1416 effort=50 velocity=2; type continuous -> revolute
- joint joint11: limit (none) -> lower=-3.1416 upper=3.1416 effort=50 velocity=2; type continuous -> revolute
- joint joint12: limit (none) -> lower=-3.1416 upper=3.1416 effort=50 velocity=2; type continuous -> revolute
- joint joint13: limit (none) -> lower=-3.1416 upper=3.1416 effort=50 velocity=2; type continuous -> revolute
- joint joint14: limit (none) -> lower=-3.1416 upper=3.1416 effort=50 velocity=2; type continuous -> revolute
- joint joint15: axis 0 0 1 -> 0 0 -1; limit (none) -> lower=-3.1416 upper=3.1416 effort=50 velocity=2; type continuous -> revolute
- joint joint16: limit (none) -> lower=-3.1416 upper=3.1416 effort=50 velocity=2; type continuous -> revolute
- joint joint17: axis 0 0 -1 -> 0 0 1; limit (none) -> lower=-3.1416 upper=3.1416 effort=50 velocity=2; type continuous -> revolute
- joint joint2: limit (none) -> lower=-3.1416 upper=3.1416 effort=50 velocity=2; type continuous -> revolute
- joint joint3: limit (none) -> lower=-3.1416 upper=3.1416 effort=50 velocity=2; type continuous -> revolute
- joint joint4: limit (none) -> lower=-3.1416 upper=3.1416 effort=50 velocity=2; type continuous -> revolute
- joint joint5: limit (none) -> lower=-3.1416 upper=3.1416 effort=50 velocity=2; type continuous -> revolute
- joint joint6: axis 0 0 1 -> 0 0 -1; limit (none) -> lower=-3.1416 upper=3.1416 effort=50 velocity=2; type continuous -> revolute
- joint joint7: limit (none) -> lower=-3.1416 upper=3.1416 effort=50 velocity=2; type continuous -> revolute

Commit message: feat:模型修改

File: src/upperlimb_robot/urdf/robot_arms.urdf (robot description, URDF)
Before this commit: robot robot_arms, 26 links, 25 joints
Joints:
- joint joint11: axis 0 0 1 -> 0 0 -1
- joint joint12: axis 0 0 1 -> 0 0 -1
- joint joint13: axis 0 0 1 -> 0 0 -1
- joint joint14: axis 0 0 1 -> 0 0 -1
